File: p-bass_wiring.sch (KiCad schematic (older format))
At the start: 5 parts

Commit message: affectation des empreintes
Parts:
- C1: footprint (none) -> Capacitors_ThroughHole:C_Disc_D6_P5
- Tone1, Volume1: footprint (none) -> Pin_Headers:Pin_Header_Straight_1x03
Changed lines of the file:
@@
 F 0 "Volume1" H 6500 3550 50  0000 C CNN
 F 1 "250k" H 6500 3650 50  0000 C CNN
-F 2 "" H 6500 3650 60  0000 C CNN
+F 2 "Pin_Headers:Pin_Header_Straight_1x03" H 6500 3650 60  0001 C CNN
 F 3 "" H 6500 3650 60  0000 C CNN
 	1    6500 3650
@@
 F 0 "Tone1" H 5850 3550 50  0000 C CNN
 F 1 "250k" H 5850 3650 50  0000 C CNN
-F 2 "" H 5850 3650 60  0000 C CNN
+F 2 "Pin_Headers:Pin_Header_Straight_1x03" H 5850 3650 60  0001 C CNN
 F 3 "" H 5850 3650 60  0000 C CNN
 	1    5850 3650
@@
 F 0 "Coil_wiring1" H 4050 3900 50  0000 C CNN
 F 1 "Switch_SPDT_x2" H 4000 3600 50  0000 C CNN
-F 2 "" H 4250 3750 60  0000 C CNN
+F 2 "" H 4250 3750 60  0001 C CNN
 F 3 "" H 4250 3750 60  0000 C CNN
 	2    4250 3750
@@
 Ground
 $Comp
-L Earth #PWR1
+L Earth #PWR01
 U 1 1 56671417
 P 6500 4050
-F 0 "#PWR1" H 6500 3800 50  0001 C CNN
+F 0 "#PWR01" H 6500 3800 50  0001 C CNN
 F 1 "Earth" H 6500 3900 50  0001 C CNN
 F 2 "" H 6500 4050 60  0000 C CNN
@@
 F 0 "Coil_wiring1" H 4050 3250 50  0000 C CNN
 F 1 "Switch_SPDT_x2" H 4000 2950 50  0000 C CNN
-F 2 "" H 4250 3100 60  0000 C CNN
+F 2 "" H 4250 3100 60  0001 C CNN
 F 3 "" H 4250 3100 60  0000 C CNN
 	1    4250 3100
@@
 F 0 "C1" H 6125 3900 50  0000 L CNN
 F 1 "0.1µ" H 6125 3700 50  0000 L CNN
-F 2 "" H 6138 3650 30  0000 C CNN
+F 2 "Capacitors_ThroughHole:C_Disc_D6_P5" H 6138 3650 30  0001 C CNN
 F 3 "" H 6100 3800 60  0000 C CNN
 	1    6100 3800
@@
 F 0 "Bypass1" H 5100 3350 50  0000 C CNN
 F 1 "Switch_SPDT_x2" H 5050 3050 50  0000 C CNN
-F 2 "" H 5300 3200 50  0000 C CNN
+F 2 "" H 5300 3200 50  0001 C CNN
 F 3 "" H 5300 3200 50  0000 C CNN
 	1    5300 3200
@@
 F 0 "Bypass1" H 6850 3700 50  0000 C CNN
 F 1 "Switch_SPDT_x2" H 6800 3400 50  0000 C CNN
-F 2 "" H 7050 3550 50  0000 C CNN
+F 2 "" H 7050 3550 50  0001 C CNN
 F 3 "" H 7050 3550 50  0000 C CNN
 	2    7050 3550
